Commit message: made the legs longer

File: stridebot.urdf (robot description, URDF)
Before this commit: robot quadruped_robot, 5 links, 4 joints
Links:
- link back_left_leg: mass 0.2 -> 0.4; geometry collision cylinder length=0.4 radius=0.05; visual cylinder length=0.4 radius=0.05
- link back_right_leg: mass 0.2 -> 0.4; geometry collision cylinder length=0.4 radius=0.05; visual cylinder length=0.4 radius=0.05
- link front_left_leg: mass 0.2 -> 0.4; geometry collision cylinder length=0.4 radius=0.05; visual cylinder length=0.4 radius=0.05
- link front_right_leg: mass 0.2 -> 0.4; geometry collision cylinder length=0.4 radius=0.05; visual cylinder length=0.4 radius=0.05
Joints:
- joint back_left_joint: origin xyz=-0.2 0.15 0 rpy=0 0 0 -> xyz=-0.2 0.15 -0.1 rpy=0 0 0
- joint back_right_joint: origin xyz=-0.2 -0.15 0 rpy=0 0 0 -> xyz=-0.2 -0.15 -0.1 rpy=0 0 0
- joint front_left_joint: origin xyz=0.2 0.15 0 rpy=0 0 0 -> xyz=0.2 0.15 -0.1 rpy=0 0 0
- joint front_right_joint: origin xyz=0.2 -0.15 0 rpy=0 0 0 -> xyz=0.2 -0.15 -0.1 rpy=0 0 0

Commit message: inconsistanly moving in need of fine tuning to reach directions exactly

File: stridebot.urdf (robot description, URDF)
Before this commit: robot quadruped_robot, 5 links, 4 joints
Joints:
- joint back_left_joint: limit effort=5.0 velocity=1.0 -> lower=-1.0 upper=1.0 effort=50.0 velocity=5.0; type continuous -> revolute
- joint back_right_joint: limit effort=5.0 velocity=1.0 -> lower=-1.0 upper=1.0 effort=50.0 velocity=5.0; type continuous -> revolute
- joint front_left_joint: limit effort=5.0 velocity=1.0 -> lower=-1.0 upper=1.0 effort=50.0 velocity=5.0; type continuous -> revolute
- joint front_right_joint: limit effort=5.0 velocity=1.0 -> lower=-1.0 upper=1.0 effort=50.0 velocity=5.0; type continuous -> revolute

Commit message: added prismatic joints to the model

File: stridebot.urdf (robot description, URDF)
Before this commit: robot quadruped_robot, 5 links, 4 joints
Links:
- added link back_left_attachment_point; visual box size=0.05 0.05 0.05
- added link back_right_attachment_point; visual box size=0.05 0.05 0.05
- added link front_left_attachment_point; visual box size=0.05 0.05 0.05
- added link front_right_attachment_point; visual box size=0.05 0.05 0.05
Joints:
- removed joint back_left_joint
- removed joint back_right_joint
- removed joint front_left_joint
- removed joint front_right_joint
- added joint back_left_prismatic: type prismatic, parent base_link, child back_left_attachment_point, origin xyz=-0.2 0.15 0 rpy=0 0 0, axis 0 0 1, limit lower=0.0 upper=0.2 effort=50.0 velocity=1.0
- added joint back_left_rotational: type continuous, parent back_left_attachment_point, child back_left_leg, origin xyz=0 0 0 rpy=0 0 0, axis 0 1 0, limit effort=5.0 velocity=1.0
- added joint back_right_prismatic: type prismatic, parent base_link, child back_right_attachment_point, origin xyz=-0.2 -0.15 0 rpy=0 0 0, axis 0 0 1, limit lower=0.0 upper=0.2 effort=50.0 velocity=1.0
- added joint back_right_rotational: type continuous, parent back_right_attachment_point, child back_right_leg, origin xyz=0 0 0 rpy=0 0 0, axis 0 1 0, limit effort=5.0 velocity=1.0
- added joint front_left_prismatic: type prismatic, parent base_link, child front_left_attachment_point, origin xyz=0.2 0.15 0 rpy=0 0 0, axis 0 0 1, limit lower=0.0 upper=0.2 effort=50.0 velocity=1.0
- added joint front_left_rotational: type continuous, parent front_left_attachment_point, child front_left_leg, origin xyz=0 0 0 rpy=0 0 0, axis 0 1 0, limit effort=5.0 velocity=1.0
- added joint front_right_prismatic: type prismatic, parent base_link, child front_right_attachment_point, origin xyz=0.2 -0.15 0 rpy=0 0 0, axis 0 0 1, limit lower=0.0 upper=0.2 effort=50.0 velocity=1.0
- added joint front_right_rotational: type continuous, parent front_right_attachment_point, child front_right_leg, origin xyz=0 0 0 rpy=0 0 0, axis 0 1 0, limit effort=5.0 velocity=1.0

Commit message: minor changes

File: stridebot.urdf (robot description, URDF)
Before this commit: robot quadruped_robot, 9 links, 8 joints
Links:
- link base_link: mass 1.0 -> 2.0
Joints:
- joint back_left_prismatic: limit lower=0.0 upper=0.2 effort=50.0 velocity=1.0 -> lower=-0.2 upper=0.2 effort=100.0 velocity=1.0
- joint back_left_rotational: limit effort=5.0 velocity=1.0 -> effort=100.0 velocity=1.0
- joint back_right_prismatic: limit lower=0.0 upper=0.2 effort=50.0 velocity=1.0 -> lower=-0.2 upper=0.2 effort=100.0 velocity=1.0
- joint back_right_rotational: limit effort=5.0 velocity=1.0 -> effort=100.0 velocity=1.0
- joint front_left_prismatic: limit lower=0.0 upper=0.2 effort=50.0 velocity=1.0 -> lower=-0.2 upper=0.2 effort=100.0 velocity=1.0
- joint front_left_rotational: limit effort=5.0 velocity=1.0 -> effort=100.0 velocity=1.0
- joint front_right_prismatic: limit lower=0.0 upper=0.2 effort=50.0 velocity=1.0 -> lower=-0.2 upper=0.2 effort=100.0 velocity=1.0
- joint front_right_rotational: limit effort=5.0 velocity=1.0 -> effort=100.0 velocity=1.0

Commit message: model can finally walk in a straight line smoothly

File: stridebot.urdf (robot description, URDF)
Before this commit: robot quadruped_robot, 9 links, 8 joints
Links:
- link back_left_leg: geometry collision cylinder length=0.3 radius=0.05; visual cylinder length=0.3 radius=0.05
- link back_right_leg: geometry collision cylinder length=0.3 radius=0.05; visual cylinder length=0.3 radius=0.05
- link base_link: geometry collision box size=0.6 0.6 0.1; visual box size=0.6 0.6 0.1
- link front_left_leg: geometry collision cylinder length=0.3 radius=0.05; visual cylinder length=0.3 radius=0.05
- link front_right_leg: geometry collision cylinder length=0.3 radius=0.05; visual cylinder length=0.3 radius=0.05
Joints:
- joint back_left_prismatic: origin xyz=-0.2 0.15 0 rpy=0 0 0 -> xyz=-0.3 0.3 0 rpy=0 0 0
- joint back_right_prismatic: origin xyz=-0.2 -0.15 0 rpy=0 0 0 -> xyz=-0.3 -0.3 0 rpy=0 0 0
- joint front_left_prismatic: origin xyz=0.2 0.15 0 rpy=0 0 0 -> xyz=0.3 0.3 0 rpy=0 0 0
- joint front_right_prismatic: origin xyz=0.2 -0.15 0 rpy=0 0 0 -> xyz=0.3 -0.3 0 rpy=0 0 0

Commit message: removed prismatic joints

File: stridebot.urdf (robot description, URDF)
Before this commit: robot quadruped_robot, 9 links, 8 joints
Links:
- removed link back_left_attachment_point
- removed link back_right_attachment_point
- removed link front_left_attachment_point
- removed link front_right_attachment_point
Joints:
- removed joint back_left_prismatic
- removed joint back_right_prismatic
- removed joint front_left_prismatic
- removed joint front_right_prismatic
- joint back_left_rotational: origin xyz=0 0 0 rpy=0 0 0 -> xyz=-0.3 0.3 -0.05 rpy=0 0 0; parent back_left_attachment_point -> base_link
- joint back_right_rotational: origin xyz=0 0 0 rpy=0 0 0 -> xyz=-0.3 -0.3 -0.05 rpy=0 0 0; parent back_right_attachment_point -> base_link
- joint front_left_rotational: origin xyz=0 0 0 rpy=0 0 0 -> xyz=0.3 0.3 -0.05 rpy=0 0 0; parent front_left_attachment_point -> base_link
- joint front_right_rotational: origin xyz=0 0 0 rpy=0 0 0 -> xyz=0.3 -0.3 -0.05 rpy=0 0 0; parent front_right_attachment_point -> base_link

Commit message: "Changed the type of join + changed the walking style"

File: stridebot.urdf (robot description, URDF)
Before this commit: robot quadruped_robot, 5 links, 4 joints
Joints:
- joint back_left_rotational: limit effort=100.0 velocity=1.0 -> lower=-0.785 upper=0.785 effort=100.0 velocity=1.0; type continuous -> revolute
- joint back_right_rotational: limit effort=100.0 velocity=1.0 -> lower=-0.785 upper=0.785 effort=100.0 velocity=1.0; type continuous -> revolute
- joint front_left_rotational: limit effort=100.0 velocity=1.0 -> lower=-0.785 upper=0.785 effort=100.0 velocity=1.0; type continuous -> revolute
- joint front_right_rotational: limit effort=100.0 velocity=1.0 -> lower=-0.785 upper=0.785 effort=100.0 velocity=1.0; type continuous -> revolute

Commit message: Funny-movement

File: stridebot.urdf (robot description, URDF)
Before this commit: robot quadruped_robot, 5 links, 4 joints
Links:
- link back_left_leg: mass 0.4 -> 5; geometry collision cylinder length=1 radius=0.05; visual cylinder length=1 radius=0.05
- link back_right_leg: mass 0.4 -> 5; geometry collision cylinder length=1 radius=0.05; visual cylinder length=1 radius=0.05
- link base_link: mass 2.0 -> 50.0
- link front_left_leg: mass 0.4 -> 5; geometry collision cylinder length=1 radius=0.05; visual cylinder length=1 radius=0.05
- link front_right_leg: mass 0.4 -> 5; geometry collision cylinder length=1 radius=0.05; visual cylinder length=1 radius=0.05

Commit message: choppy but working model with prismatic joints

File: stridebot.urdf (robot description, URDF)
Before this commit: robot quadruped_robot, 5 links, 4 joints
Links:
- added link back_left_rotational_link, mass 0.1
- added link back_right_rotational_link, mass 0.1
- added link front_left_rotational_link, mass 0.1
- added link front_right_rotational_link, mass 0.1
Joints:
- added joint back_left_prismatic: type prismatic, parent base_link, child back_left_rotational_link, origin xyz=-0.3 0.3 0.0 rpy=0 0 0, axis 0 0 1, limit lower=0 upper=0.1 effort=100.0 velocity=1.0
- added joint back_right_prismatic: type prismatic, parent base_link, child back_right_rotational_link, origin xyz=-0.3 -0.3 0.0 rpy=0 0 0, axis 0 0 1, limit lower=0 upper=0.1 effort=100.0 velocity=1.0
- added joint front_left_prismatic: type prismatic, parent base_link, child front_left_rotational_link, origin xyz=0.3 0.3 0.0 rpy=0 0 0, axis 0 0 1, limit lower=0 upper=0.1 effort=100.0 velocity=1.0
- added joint front_right_prismatic: type prismatic, parent base_link, child front_right_rotational_link, origin xyz=0.3 -0.3 0.0 rpy=0 0 0, axis 0 0 1, limit lower=0 upper=0.1 effort=100.0 velocity=1.0
- joint back_left_rotational: origin xyz=-0.3 0.3 -0.05 rpy=0 0 0 -> xyz=0 0 -0.05 rpy=0 0 0; parent base_link -> back_left_rotational_link
- joint back_right_rotational: origin xyz=-0.3 -0.3 -0.05 rpy=0 0 0 -> xyz=0 0 -0.05 rpy=0 0 0; parent base_link -> back_right_rotational_link
- joint front_left_rotational: origin xyz=0.3 0.3 -0.05 rpy=0 0 0 -> xyz=0 0 -0.05 rpy=0 0 0; parent base_link -> front_left_rotational_link
- joint front_right_rotational: origin xyz=0.3 -0.3 -0.05 rpy=0 0 0 -> xyz=0 0 -0.05 rpy=0 0 0; parent base_link -> front_right_rotational_link

Commit message: a bit smoother now

File: stridebot.urdf (robot description, URDF)
Before this commit: robot quadruped_robot, 9 links, 8 joints
Links:
- link base_link: mass 50.0 -> 5.0

Commit message: smooth walking forward motion

File: stridebot.urdf (robot description, URDF)
Before this commit: robot quadruped_robot, 9 links, 8 joints
Links:
- link back_left_leg: geometry collision cylinder length=0.6 radius=0.05; visual cylinder length=0.6 radius=0.05
- link back_right_leg: geometry collision cylinder length=0.6 radius=0.05; visual cylinder length=0.6 radius=0.05
- link front_left_leg: geometry collision cylinder length=0.6 radius=0.05; visual cylinder length=0.6 radius=0.05
- link front_right_leg: geometry collision cylinder length=0.6 radius=0.05; visual cylinder length=0.6 radius=0.05
Joints:
- joint back_left_prismatic: origin xyz=-0.3 0.3 0.0 rpy=0 0 0 -> xyz=-0.3 0.3 -0.2 rpy=0 0 0
- joint back_right_prismatic: origin xyz=-0.3 -0.3 0.0 rpy=0 0 0 -> xyz=-0.3 -0.3 -0.2 rpy=0 0 0
- joint front_left_prismatic: origin xyz=0.3 0.3 0.0 rpy=0 0 0 -> xyz=0.3 0.3 -0.2 rpy=0 0 0
- joint front_right_prismatic: origin xyz=0.3 -0.3 0.0 rpy=0 0 0 -> xyz=0.3 -0.3 -0.2 rpy=0 0 0

Commit message: adjusted base link mass

File: stridebot.urdf (robot description, URDF)
Before this commit: robot quadruped_robot, 9 links, 8 joints
Links:
- link base_link: mass 5.0 -> 40.0
